Commit message: 解决了MoveIt轨迹离线控制存在角度换算的错误

File: install/so_arm100/share/so_arm100/urdf/so_arm100.urdf.xacro (robot description, xacro)
@@ -1 +1,73 @@
-/home/ubuntu22/ros2_so_arm100/so_arm100/urdf/so_arm100.urdf.xacro
+<?xml version="1.0"?>
+<robot xmlns:xacro="http://www.ros.org/wiki/xacro" name="so_arm100">
+    <xacro:arg name="prefix" default=""/>
+    <xacro:arg name="hardware_type" default="mock_components"/>
+    <!-- Import main macro -->
+    <xacro:include filename="$(find so_arm100)/urdf/so_arm100_macro.xacro"/>
+    <!-- Create robot by calling main macro -->
+    <xacro:so_arm100 prefix="$(arg prefix)"/>
+    <ros2_control name="so_arm100_system" type="system">
+        <hardware>
+            <xacro:if value="${'$(arg hardware_type)' == 'mock_components'}">
+                <plugin>mock_components/GenericSystem</plugin>
+            </xacro:if>
+            <xacro:if value="${'$(arg hardware_type)' == 'real'}">
+                <plugin>feetech_ros2_driver/FeetechHardwareInterface</plugin>
+                <param name="usb_port">/dev/LeRobotFollower</param>
+            </xacro:if>
+        </hardware>
+        <joint name="shoulder_pan_joint">
+            <param name="id">1</param>
+            <param name="offset">2048</param>
+            <param name="p_coefficient">8</param>
+            <command_interface name="position"/>
+            <state_interface name="position"/>
+            <state_interface name="velocity"/>
+        </joint>
+        <joint name="shoulder_lift_joint">
+            <param name="id">2</param>
+            <param name="offset">2125</param>
+            <param name="p_coefficient">16</param>
+            <command_interface name="position"/>
+            <state_interface name="position"/>
+            <state_interface name="velocity"/>
+        </joint>
+        <joint name="elbow_joint">
+            <param name="id">3</param>
+            <param name="offset">2080</param>
+            <param name="p_coefficient">16</param>
+            <command_interface name="position"/>
+            <state_interface name="position"/>
+            <state_interface name="velocity"/>
+        </joint>
+        <joint name="wrist_pitch_joint">
+            <param name="id">4</param>
+            <param name="offset">3110</param>
+            <param name="p_coefficient">16</param>
+            <command_interface name="position"/>
+            <state_interface name="position"/>
+            <state_interface name="velocity"/>
+        </joint>
+        <joint name="wrist_roll_joint">
+            <param name="id">5</param>
+            <param name="offset">2048</param>
+            <param name="p_coefficient">16</param>
+            <command_interface name="position"/>
+            <state_interface name="position"/>
+            <state_interface name="velocity"/>
+        </joint>
+        <joint name="jaw_joint">
+            <param name="id">6</param>
+            <param name="offset">2048</param>
+            <param name="p_coefficient">16</param>
+            <command_interface name="position"/>
+            <state_interface name="position"/>
+            <state_interface name="velocity"/>
+        </joint>
+    </ros2_control>
+    <gazebo>
+        <plugin name="gazebo_ros2_control" filename="libgazebo_ros2_control.so">
+            <parameters>$(find so_arm100_moveit_config)/config/controllers.yaml</parameters>
+        </plugin>
+    </gazebo>
+</robot>

File: install/so_arm100/share/so_arm100/urdf/so_arm100_control.urdf.xacro (robot description, xacro)
@@ -1 +1,53 @@
-/home/ubuntu22/ros2_so_arm100/so_arm100/urdf/so_arm100_control.urdf.xacro
+<?xml version="1.0"?>
+<robot xmlns:xacro="http://www.ros.org/wiki/xacro" name="so_arm100">
+    <!-- Import the original URDF -->
+    <xacro:include filename="$(find so_arm100)/urdf/so_arm100.urdf"/>
+    <!-- ros2_control plugin -->
+    <xacro:macro name="so_arm100_ros2_control">
+        <ros2_control name="so_arm100_system" type="system">
+            <hardware>
+                <plugin>mock_components/GenericSystem</plugin>
+            </hardware>
+            <!-- Arm joints -->
+            <joint name="shoulder_pan_joint">
+                <command_interface name="position"/>
+                <state_interface name="position"/>
+                <state_interface name="velocity"/>
+            </joint>
+            <joint name="shoulder_lift_joint">
+                <command_interface name="position"/>
+                <state_interface name="position"/>
+                <state_interface name="velocity"/>
+            </joint>
+            <joint name="elbow_joint">
+                <command_interface name="position"/>
+                <state_interface name="position"/>
+                <state_interface name="velocity"/>
+            </joint>
+            <joint name="wrist_pitch_joint">
+                <command_interface name="position"/>
+                <state_interface name="position"/>
+                <state_interface name="velocity"/>
+            </joint>
+            <joint name="wrist_roll_joint">
+                <command_interface name="position"/>
+                <state_interface name="position"/>
+                <state_interface name="velocity"/>
+            </joint>
+            <!-- Gripper joint -->
+            <joint name="jaw_joint">
+                <command_interface name="position"/>
+                <state_interface name="position"/>
+                <state_interface name="velocity"/>
+            </joint>
+        </ros2_control>
+        <!-- Gazebo plugin for ros2_control -->
+        <gazebo>
+            <plugin name="gazebo_ros2_control" filename="libgazebo_ros2_control.so">
+                <parameters>$(find so_arm100_moveit_config)/config/ros2_controllers.yaml</parameters>
+            </plugin>
+        </gazebo>
+    </xacro:macro>
+    <!-- Include the ros2_control macro -->
+    <xacro:so_arm100_ros2_control/>
+</robot>

File: install/so_arm100/share/so_arm100/urdf/so_arm100_macro.xacro (robot description, xacro)
@@ -1 +1,6 @@
-/home/ubuntu22/ros2_so_arm100/so_arm100/urdf/so_arm100_macro.xacro
+<?xml version="1.0"?>
+<robot xmlns:xacro="http://www.ros.org/wiki/xacro">
+    <xacro:macro name="so_arm100" params="prefix">
+        <xacro:include filename="$(find so_arm100)/urdf/so_arm100.urdf"/>
+    </xacro:macro>
+</robot>
